Commit message: sync

File: robots/alexandros.urdf.xacro (robot description, xacro)
@@ -6,4 +6,5 @@
     <!-- Initialize Panda -->
     <xacro:arg name="arm_id" default="panda" />
+    <xacro:arg name="hand" default="true" />
     <xacro:franka_robot arm_id="$(arg arm_id)"
                         joint_limits="${xacro.load_yaml('$(find franka_description)/robots/panda/joint_limits.yaml')}">
@@ -11,6 +12,7 @@
     <!-- Initialize the Joint between Ridgeback and Panda -->
     <joint name="panda_joint" type="fixed">
-        <parent link="panda_link0"/>
-        <child link="base_link"/>
-        <origin xyz="0 0 0" rpy="0 0 0"/>
+        <origin xyz="0 0 0.3" rpy="0 0 0"/>
+        <parent link="base_link"/>
+        <child link="panda_link0"/>
+    </joint>
 </robot>

Commit message: sync

File: robots/alexandros.urdf.xacro (robot description, xacro)
@@ -4,5 +4,6 @@
     <xacro:include filename="$(find franka_description)/robots/common/franka_robot.xacro"/>
     <xacro:include filename="$(find ridgeback_description)/urdf/ridgeback.urdf.xacro"/>
-    <!-- TODO: Add Realsense Camer -->
+    <xacro:arg name="use_nominal_extrinsics" default="false"/>
+    <xacro:include filename="$(find realsense2_description)/urdf/_d455.urdf.xacro" />
     <!-- Initialize Panda -->
     <xacro:arg name="arm_id" default="panda" />
@@ -17,3 +18,7 @@
         <child link="panda_link0"/>
     </joint>
+    <!-- Add Camera -->
+    <xacro:sensor_d455 parent="panda_hand" use_nominal_extrinsics="$(arg use_nominal_extrinsics)">
+    <origin xyz="0.09 0 0" rpy="0 0 0"/>
+  </xacro:sensor_d455>
 </robot>

Commit message: sync urdf

File: robots/alexandros.urdf.xacro (robot description, xacro)
@@ -14,5 +14,5 @@
     <!-- Initialize the Joint between Ridgeback and Panda -->
     <joint name="panda_joint" type="fixed">
-        <origin xyz="0 0 0.3" rpy="0 0 0"/>
+        <origin xyz="0 0 0.7112" rpy="0 0 0"/>
         <parent link="base_link"/>
         <child link="panda_link0"/>
@@ -20,5 +20,5 @@
     <!-- Add Camera -->
     <xacro:sensor_d455 parent="panda_hand" use_nominal_extrinsics="$(arg use_nominal_extrinsics)">
-    <origin xyz="0.09 0 0" rpy="0 0 0"/>
+    <origin xyz="0.05 0 0" rpy="0 -1.57 0"/>
   </xacro:sensor_d455>
 </robot>

Commit message: Adjust spacing

File: robots/alexandros.urdf.xacro (robot description, xacro)
@@ -1,23 +1,23 @@
 <?xml version='1.0' encoding='utf-8'?>
 <robot xmlns:xacro="http://www.ros.org/wiki/xacro" name="alexandros">
-    <!-- Include the robots -->
-    <xacro:include filename="$(find franka_description)/robots/common/franka_robot.xacro"/>
-    <xacro:include filename="$(find ridgeback_description)/urdf/ridgeback.urdf.xacro"/>
-    <xacro:arg name="use_nominal_extrinsics" default="false"/>
-    <xacro:include filename="$(find realsense2_description)/urdf/_d455.urdf.xacro" />
-    <!-- Initialize Panda -->
-    <xacro:arg name="arm_id" default="panda" />
-    <xacro:arg name="hand" default="true" />
-    <xacro:franka_robot arm_id="$(arg arm_id)"
-                        joint_limits="${xacro.load_yaml('$(find franka_description)/robots/panda/joint_limits.yaml')}">
-    </xacro:franka_robot>
-    <!-- Initialize the Joint between Ridgeback and Panda -->
-    <joint name="panda_joint" type="fixed">
-        <origin xyz="0 0 0.7112" rpy="0 0 0"/>
-        <parent link="base_link"/>
-        <child link="panda_link0"/>
-    </joint>
-    <!-- Add Camera -->
-    <xacro:sensor_d455 parent="panda_hand" use_nominal_extrinsics="$(arg use_nominal_extrinsics)">
+  <!-- Include the robots -->
+  <xacro:include filename="$(find franka_description)/robots/common/franka_robot.xacro"/>
+  <xacro:include filename="$(find ridgeback_description)/urdf/ridgeback.urdf.xacro"/>
+  <xacro:arg name="use_nominal_extrinsics" default="false"/>
+  <xacro:include filename="$(find realsense2_description)/urdf/_d455.urdf.xacro" />
+  <!-- Initialize Panda -->
+  <xacro:arg name="arm_id" default="panda" />
+  <xacro:arg name="hand" default="true" />
+  <xacro:franka_robot arm_id="$(arg arm_id)"
+                      joint_limits="${xacro.load_yaml('$(find franka_description)/robots/panda/joint_limits.yaml')}">
+  </xacro:franka_robot>
+  <!-- Initialize the Joint between Ridgeback and Panda -->
+  <joint name="panda_joint" type="fixed">
+    <origin xyz="0 0 0.7112" rpy="0 0 0"/>
+    <parent link="base_link"/>
+    <child link="panda_link0"/>
+  </joint>
+  <!-- Add Camera -->
+  <xacro:sensor_d455 parent="panda_hand" use_nominal_extrinsics="$(arg use_nominal_extrinsics)">
     <origin xyz="0.05 0 0" rpy="0 -1.57 0"/>
   </xacro:sensor_d455>
